Commit message: Sprint 3 completed: ros2_control, diff drive, odometry

File: src/amr_description/urdf/amr_caster.xacro (robot description, xacro)
@@ -2,6 +2,6 @@
 <robot xmlns:xacro="http://www.ros.org/wiki/xacro">
   <xacro:property name="caster_roll" value="1.57079632679"/>
-  <xacro:macro name="amr_caster">
-    <link name="caster_link">
+  <xacro:macro name="caster_wheel" params="link_name joint_name x_offset">
+    <link name="${link_name}">
       <visual>
         <origin xyz="0 0 0" rpy="${caster_roll} 0 0"/>
@@ -29,11 +29,15 @@
       </inertial>
     </link>
-    <joint name="caster_joint" type="fixed">
+    <joint name="${joint_name}" type="fixed">
       <parent link="base_link"/>
-      <child link="caster_link"/>
+      <child link="${link_name}"/>
       <origin
-        xyz="${caster_x_offset} ${caster_y_offset} ${caster_z_offset}"
+        xyz="${x_offset} ${caster_y_offset} ${caster_z_offset}"
         rpy="0 0 0"/>
     </joint>
   </xacro:macro>
+  <xacro:macro name="amr_caster">
+    <xacro:caster_wheel link_name="caster_link" joint_name="caster_joint" x_offset="${caster_x_offset}"/>
+    <xacro:caster_wheel link_name="rear_caster_link" joint_name="rear_caster_joint" x_offset="${-caster_x_offset}"/>
+  </xacro:macro>
 </robot>

File: src/amr_description/urdf/amr_properties.xacro (robot description, xacro)
@@ -23,5 +23,6 @@
   <xacro:property name="caster_x_offset" value="0.180"/>
   <xacro:property name="caster_y_offset" value="0.000"/>
-  <xacro:property name="caster_z_offset" value="${wheel_z_offset}"/>
+  <!-- Align caster ground contact with drive wheels (smaller radius → lower joint z) -->
+  <xacro:property name="caster_z_offset" value="${wheel_z_offset - wheel_radius + caster_radius}"/>
   <!-- Sensors (mount poses relative to base_link) -->
   <xacro:property name="laser_x_offset" value="0.000"/>

File: src/amr_description/urdf/amr_wheels.xacro (robot description, xacro)
@@ -2,5 +2,5 @@
 <robot xmlns:xacro="http://www.ros.org/wiki/xacro">
   <xacro:property name="wheel_roll" value="1.57079632679"/>
-  <xacro:macro name="drive_wheel" params="prefix y_offset">
+  <xacro:macro name="drive_wheel" params="prefix y_offset axis_dir:=1">
     <link name="${prefix}_wheel_link">
       <visual>
@@ -35,10 +35,10 @@
         xyz="${wheel_x_offset} ${y_offset} ${wheel_z_offset}"
         rpy="0 0 0"/>
-      <axis xyz="0 1 0"/>
+      <axis xyz="0 ${axis_dir} 0"/>
     </joint>
   </xacro:macro>
   <xacro:macro name="amr_wheels">
-    <xacro:drive_wheel prefix="left" y_offset="${wheel_separation / 2.0}"/>
-    <xacro:drive_wheel prefix="right" y_offset="${-wheel_separation / 2.0}"/>
+    <xacro:drive_wheel prefix="left" y_offset="${wheel_separation / 2.0}" axis_dir="1"/>
+    <xacro:drive_wheel prefix="right" y_offset="${-wheel_separation / 2.0}" axis_dir="1"/>
   </xacro:macro>
 </robot>

File: src/amr_gazebo/urdf/amr.gazebo.xacro (robot description, xacro)
@@ -10,11 +10,26 @@
   <xacro:include filename="$(find amr_description)/urdf/amr_caster.xacro"/>
   <xacro:include filename="$(find amr_description)/urdf/amr_sensors.xacro"/>
+  <xacro:include filename="$(find amr_description)/urdf/amr_ros2_control.xacro"/>
   <xacro:include filename="$(find amr_gazebo)/urdf/amr_lidar.gazebo.xacro"/>
   <xacro:include filename="$(find amr_gazebo)/urdf/amr_imu.gazebo.xacro"/>
+  <xacro:include filename="$(find amr_gazebo)/urdf/amr_base.gazebo.xacro"/>
+  <xacro:include filename="$(find amr_gazebo)/urdf/amr_wheels.gazebo.xacro"/>
+  <xacro:include filename="$(find amr_gazebo)/urdf/amr_caster.gazebo.xacro"/>
   <xacro:amr_base/>
   <xacro:amr_wheels/>
   <xacro:amr_caster/>
   <xacro:amr_sensors/>
+  <xacro:amr_ros2_control/>
   <xacro:amr_lidar_gazebo/>
   <xacro:amr_imu_gazebo/>
+  <xacro:amr_base_gazebo/>
+  <xacro:amr_wheels_gazebo/>
+  <xacro:amr_caster_gazebo/>
+  <gazebo>
+    <plugin filename="libgazebo_ros2_control.so" name="gazebo_ros2_control">
+      <robot_param>robot_description</robot_param>
+      <robot_param_node>robot_state_publisher</robot_param_node>
+      <parameters>$(find amr_control)/config/ros2_control.yaml</parameters>
+    </plugin>
+  </gazebo>
 </robot>
