Commit message: Sprint 7 Phase 1: integrate RGB camera and restore AMR regression

File: src/amr_description/urdf/amr_properties.xacro (robot description, xacro)
@@ -37,4 +37,13 @@
   <xacro:property name="imu_size" value="0.030"/>
   <xacro:property name="imu_mass" value="0.010"/>
+  <!-- RGB camera: front of chassis, z≈0.25 m on base_link (Sprint 7 spec) -->
+  <xacro:property name="camera_x_offset" value="0.250"/>
+  <xacro:property name="camera_y_offset" value="0.000"/>
+  <xacro:property name="camera_z_offset" value="0.250"/>
+  <xacro:property name="camera_width" value="0.040"/>
+  <xacro:property name="camera_height" value="0.030"/>
+  <xacro:property name="camera_depth" value="0.025"/>
+  <xacro:property name="camera_mass" value="0.050"/>
+  <xacro:property name="camera_lens_x" value="0.0125"/>
   <!-- Derived: base_link height so wheel contact meets ground at base_footprint -->
   <xacro:property name="base_link_z" value="${wheel_radius - wheel_z_offset}"/>
@@ -54,3 +63,6 @@
     <color rgba="0.20 0.40 0.80 1.0"/>
   </material>
+  <material name="camera_grey">
+    <color rgba="0.25 0.25 0.28 1.0"/>
+  </material>
 </robot>

File: src/amr_description/urdf/amr_sensors.xacro (robot description, xacro)
@@ -70,4 +70,45 @@
         rpy="0 0 0"/>
     </joint>
+    <!-- RGB camera mount (x forward on base_link) -->
+    <link name="camera_link">
+      <visual>
+        <origin xyz="${camera_lens_x} 0 0" rpy="0 0 0"/>
+        <geometry>
+          <box size="${camera_depth} ${camera_width} ${camera_height}"/>
+        </geometry>
+        <material name="camera_grey"/>
+      </visual>
+      <collision>
+        <origin xyz="${camera_lens_x} 0 0" rpy="0 0 0"/>
+        <geometry>
+          <box size="${camera_depth} ${camera_width} ${camera_height}"/>
+        </geometry>
+      </collision>
+      <inertial>
+        <origin xyz="${camera_lens_x} 0 0" rpy="0 0 0"/>
+        <mass value="${camera_mass}"/>
+        <inertia
+          ixx="${camera_mass / 12.0 * (camera_width * camera_width + camera_height * camera_height)}"
+          ixy="0.0"
+          ixz="0.0"
+          iyy="${camera_mass / 12.0 * (camera_depth * camera_depth + camera_height * camera_height)}"
+          iyz="0.0"
+          izz="${camera_mass / 12.0 * (camera_depth * camera_depth + camera_width * camera_width)}"/>
+      </inertial>
+    </link>
+    <joint name="camera_joint" type="fixed">
+      <parent link="base_link"/>
+      <child link="camera_link"/>
+      <origin
+        xyz="${camera_x_offset} ${camera_y_offset} ${camera_z_offset}"
+        rpy="0 0 0"/>
+    </joint>
+    <!-- REP-103 optical frame - z forward, x right, y down -->
+    <link name="camera_optical_frame"/>
+    <joint name="camera_optical_joint" type="fixed">
+      <parent link="camera_link"/>
+      <child link="camera_optical_frame"/>
+      <origin xyz="0 0 0" rpy="-1.57079632679 0 -1.57079632679"/>
+    </joint>
   </xacro:macro>
 </robot>

File: src/amr_gazebo/urdf/amr.gazebo.xacro (robot description, xacro)
@@ -5,4 +5,7 @@
 -->
 <robot xmlns:xacro="http://www.ros.org/wiki/xacro" name="amr">
+  <!-- Absolute path passed from gazebo.launch.py (avoids unresolved $(find) in gzserver). -->
+  <xacro:arg name="ros2_control_config" default="$(find amr_control)/config/ros2_control.yaml"/>
+  <xacro:property name="ros2_control_config" value="$(arg ros2_control_config)"/>
   <xacro:include filename="$(find amr_description)/urdf/amr_properties.xacro"/>
   <xacro:include filename="$(find amr_description)/urdf/amr_base.xacro"/>
@@ -13,7 +16,9 @@
   <xacro:include filename="$(find amr_gazebo)/urdf/amr_lidar.gazebo.xacro"/>
   <xacro:include filename="$(find amr_gazebo)/urdf/amr_imu.gazebo.xacro"/>
+  <xacro:include filename="$(find amr_gazebo)/urdf/amr_camera.gazebo.xacro"/>
   <xacro:include filename="$(find amr_gazebo)/urdf/amr_base.gazebo.xacro"/>
   <xacro:include filename="$(find amr_gazebo)/urdf/amr_wheels.gazebo.xacro"/>
   <xacro:include filename="$(find amr_gazebo)/urdf/amr_caster.gazebo.xacro"/>
+  <xacro:include filename="$(find amr_gazebo)/urdf/amr_ros2_control.gazebo.xacro"/>
   <xacro:amr_base/>
   <xacro:amr_wheels/>
@@ -23,13 +28,8 @@
   <xacro:amr_lidar_gazebo/>
   <xacro:amr_imu_gazebo/>
+  <xacro:amr_camera_gazebo/>
   <xacro:amr_base_gazebo/>
   <xacro:amr_wheels_gazebo/>
   <xacro:amr_caster_gazebo/>
-  <gazebo>
-    <plugin filename="libgazebo_ros2_control.so" name="gazebo_ros2_control">
-      <robot_param>robot_description</robot_param>
-      <robot_param_node>robot_state_publisher</robot_param_node>
-      <parameters>$(find amr_control)/config/ros2_control.yaml</parameters>
-    </plugin>
-  </gazebo>
+  <xacro:amr_ros2_control_gazebo/>
 </robot>
